Commit message: Fixes warnings

File: ackermann_vehicle_description/urdf/augmented_rc_car.urdf.xacro (robot description, xacro)
@@ -203,5 +203,7 @@
     <transmission name="${lr_prefix}_${fr_prefix}_shock_trans">
       <type>transmission_interface/SimpleTransmission</type>
-      <joint name="${lr_prefix}_${fr_prefix}_shock"/>
+      <joint name="${lr_prefix}_${fr_prefix}_shock">
+        <hardwareInterface>hardware_interface/EffortJointInterface</hardwareInterface>
+      </joint>
       <actuator name="${lr_prefix}_${fr_prefix}_shock_act">
         <hardwareInterface>EffortJointInterface</hardwareInterface>
@@ -226,5 +228,7 @@
     <transmission name="${lr_prefix}_${fr_prefix}_axle_trans">
       <type>transmission_interface/SimpleTransmission</type>
-      <joint name="${lr_prefix}_${fr_prefix}_axle"/>
+      <joint name="${lr_prefix}_${fr_prefix}_axle">
+        <hardwareInterface>hardware_interface/EffortJointInterface</hardwareInterface>
+      </joint>
       <actuator name="${lr_prefix}_${fr_prefix}_axle_act">
         <hardwareInterface>EffortJointInterface</hardwareInterface>
@@ -278,5 +282,7 @@
     <transmission name="${lr_prefix}_steering_trans">
       <type>transmission_interface/SimpleTransmission</type>
-      <joint name="${lr_prefix}_steering_joint"/>
+      <joint name="${lr_prefix}_steering_joint">
+        <hardwareInterface>hardware_interface/EffortJointInterface</hardwareInterface>
+      </joint>
       <actuator name="${lr_prefix}_steering_act">
         <hardwareInterface>EffortJointInterface</hardwareInterface>
